File: hw/zumo_uni_i2c_01.brd (EAGLE design)
At the start: 100 x 80 mm, 6 parts

Commit message: added
Parts:
- added 1, 10, 2, 3, 4, 5, 6, 7, 8, 9: (no value), wirepad:SMD1,27-2,54
- added C1: (no value), rcl:C0805
- added C2: (no value), rcl:SMC_C
- added CLK, GND, INT, M1, M10, M11, M12, M13, M14, M15, M16, M2, M3, M4, M5, M6, M7, M8, M9, MISO1, MISO10, MISO11, MISO12, MISO13, MISO14, MISO15, MISO16, MISO17, MISO18, MISO19, MISO20, MISO21, MISO22, MISO23, MISO24, MISO25, MISO26, MISO27, MISO28, MISO29, MISO30, MISO31, MISO32, MISO33, MISO34, MISO35, MISO36, MISO37, MISO4, MISO41, MISO43, MISO5, MISO6, MISO7, MISO8, MISO9, PAD10, PAD11, PAD12, PAD13, PAD14, PAD15, PAD16, PAD17, PAD18, PAD19, PAD20, PAD21, PAD22, PAD23, PAD24, PAD25, PAD26, PAD27, PAD28, PAD29, PAD30, PAD31, PAD32, PAD33, PAD34, PAD35, PAD36, PAD37, PAD38, PAD39, PAD40, PAD41, PAD42, PAD43, PAD44, PAD45, PAD46, PAD47, PAD48, PAD49, PAD50, PAD51, PAD52, PAD53, PAD54, PAD55, PAD56, PAD57, PAD58, PAD59, PAD60, PAD61, PAD62, PAD63, PAD64, PAD65, PAD66, PAD67, PAD68, PAD69, PAD7, PAD70, PAD71, PAD72, PAD73, PAD74, PAD75, PAD76, PAD77, PAD78, PAD79, PAD8, PAD80, PAD81, PAD82, PAD83, PAD84, PAD85, PAD86, PAD87, PAD88, PAD89, PAD9, PAD90, PAD91, PAD92, PAD93, PAD94, PAD95, PAD96, RESET, SCL, SDA, U33, U5, UCH: (no value), wirepad:1,6/0,9
- added H1: MOUNT-HOLE3.2, holes:3,2
- added IC1: TINY24/44/84-SSU, avr-7:SOIC14
- added L_GND, L_GPIO1, L_SCL, L_SDA, L_VCC, L_XSHUT, M1A, M1B, M2A, M2B: (no value), wirepad:1,6/0,8
- added R1, R2: (no value), rcl:M0805
- added SJ1, SJ2, SJ3: (no value), jumper:SJ
- added SV1: (no value), con-harting-ml:ML6
- added SV2: (no value), con-lstb:MA04-1
- PAD1, PAD2, PAD3, PAD4, PAD5, PAD6: device wirepad:SMD1,27-2,54 -> wirepad:1,6/0,9
- moved PAD5 63.4 mm to (11.4, 72.4)
- moved PAD4 58.2 mm to (8.89, 72.4)
- moved PAD2 55.1 mm to (19.1, 62.2)
- moved PAD3 53.6 mm to (8.89, 69.8)
- moved PAD1 47.8 mm to (19.1, 52.1)
- moved PAD6 38.8 mm to (19.1, 64.8)
Connections:
- removed net SPI_CLK: PAD3.1
- removed net SPI_CS: PAD5.1
- removed net SPI_MISO: PAD1.1
- removed net SPI_MOSI: PAD4.1
- new net 1A: M12.1, M1A.1
- new net 1B: M11.1, M1B.1
- new net 2A: M13.1, M2A.1
- new net 2B: M14.1, M2B.1
- new net FON: 3.1, CLK.1
- new net GPIO1: IC1.3, L_GPIO1.1
- new net INT: 9.1, IC1.8, INT.1, SV1.1
- new net M_DIR: IC1.12, M8.1
- new net M_EN: IC1.2, M1.1
- new net M_MS1: M2.1, SJ1.2
- new net M_MS2: M3.1, SJ2.2
- new net M_MS3: M4.1, SJ3.2
- new net M_RESET: IC1.6, M5.1
- new net M_SLEEP: IC1.10, M6.1
- new net M_STEP: IC1.11, M7.1
- new net N$9: IC1.13, R1.2, R2.2
- new net RESET: 5.1, IC1.4, RESET.1, SV1.5
- new net SCL: 7.1, IC1.9, L_SCL.1, MISO41.1, SCL.1, SV1.3, SV2.2
- new net SDA: 1.1, IC1.7, L_SDA.1, MISO21.1, SDA.1, SV1.4, SV2.1
- new net U5: 4.1, C2.+, M16.1, R2.1, U5.1
- new net UCH: 6.1, UCH.1
- new net XSHUT: IC1.5, L_XSHUT.1
- net GND: now also 10.1, 8.1, C1.2, C2.-, GND.1, IC1.14, L_GND.1, M15.1, M9.1, MISO1.1, MISO10.1, MISO11.1, MISO12.1, MISO13.1, MISO14.1, MISO15.1, MISO16.1, MISO17.1, MISO18.1, MISO19.1, MISO20.1, MISO43.1, MISO5.1, MISO6.1, MISO7.1, MISO8.1, MISO9.1, R1.1, SV1.6, SV2.4; no longer PAD6.1
- net U3.3: now also 2.1, C1.1, IC1.1, L_VCC.1, M10.1, MISO22.1, MISO23.1, MISO24.1, MISO25.1, MISO26.1, MISO27.1, MISO28.1, MISO29.1, MISO30.1, MISO31.1, MISO32.1, MISO33.1, MISO34.1, MISO35.1, MISO36.1, MISO37.1, MISO4.1, SJ1.1, SJ2.1, SJ3.1, SV1.2, SV2.3, U33.1; no longer PAD2.1
Routing:
- net U3.3: track 0.00 -> 115.6 mm, vias 0 -> 5
- net SDA: track 0.00 -> 91.8 mm, vias 0 -> 3
- net GND: track 0.00 -> 89.9 mm
- net 1B: track 0.00 -> 81.6 mm, vias 0 -> 1
- net 1A: track 0.00 -> 80.4 mm
- net SCL: track 0.00 -> 75.4 mm, vias 0 -> 1
- net 2B: track 0.00 -> 74.9 mm, vias 0 -> 1
- net 2A: track 0.00 -> 72.3 mm, vias 0 -> 1
- net XSHUT: track 0.00 -> 67.0 mm, vias 0 -> 1
- net GPIO1: track 0.00 -> 63.6 mm, vias 0 -> 1
- net UCH: track 0.00 -> 63.4 mm, vias 0 -> 2
- net M_EN: track 0.00 -> 52.5 mm, vias 0 -> 1
- net U5: track 0.00 -> 12.7 mm
- net RESET: track 0.00 -> 8.67 mm, vias 0 -> 1
- net N$9: track 0.00 -> 8.01 mm
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Other:
- board size 100 x 80 mm -> 21.6 x 90.2 mm
