File: hw/zumo_uni_i2c_01.sch (EAGLE design)
At the start: 6 parts

Commit message: added
Parts:
- added 1, 10, 2, 3, 4, 5, 6, 7, 8, 9: (no value), wirepad:SMD2
- added C1: (no value), rcl:C-EUC0805
- added C2: (no value), rcl:CPOL-EUSMCC
- added CLK, GND, INT, M1, M10, M11, M12, M13, M14, M15, M16, M2, M3, M4, M5, M6, M7, M8, M9, MISO1, MISO10, MISO11, MISO12, MISO13, MISO14, MISO15, MISO16, MISO17, MISO18, MISO19, MISO20, MISO21, MISO22, MISO23, MISO24, MISO25, MISO26, MISO27, MISO28, MISO29, MISO30, MISO31, MISO32, MISO33, MISO34, MISO35, MISO36, MISO37, MISO4, MISO41, MISO43, MISO5, MISO6, MISO7, MISO8, MISO9, PAD10, PAD11, PAD12, PAD13, PAD14, PAD15, PAD16, PAD17, PAD18, PAD19, PAD20, PAD21, PAD22, PAD23, PAD24, PAD25, PAD26, PAD27, PAD28, PAD29, PAD30, PAD31, PAD32, PAD33, PAD34, PAD35, PAD36, PAD37, PAD38, PAD39, PAD40, PAD41, PAD42, PAD43, PAD44, PAD45, PAD46, PAD47, PAD48, PAD49, PAD50, PAD51, PAD52, PAD53, PAD54, PAD55, PAD56, PAD57, PAD58, PAD59, PAD60, PAD61, PAD62, PAD63, PAD64, PAD65, PAD66, PAD67, PAD68, PAD69, PAD7, PAD70, PAD71, PAD72, PAD73, PAD74, PAD75, PAD76, PAD77, PAD78, PAD79, PAD8, PAD80, PAD81, PAD82, PAD83, PAD84, PAD85, PAD86, PAD87, PAD88, PAD89, PAD9, PAD90, PAD91, PAD92, PAD93, PAD94, PAD95, PAD96, RESET, SCL, SDA, U33, U5, UCH: (no value), wirepad:1,6/0,9
- added H1: MOUNT-HOLE3.2, holes:MOUNT-HOLE3.2
- added IC1: TINY24/44/84-SSU, avr-7:TINY24/44/84-SSU
- added L_GND, L_GPIO1, L_SCL, L_SDA, L_VCC, L_XSHUT, M1A, M1B, M2A, M2B: (no value), wirepad:1,6/0,8
- added R1, R2: (no value), rcl:R-EU_M0805
- added SJ1, SJ2, SJ3: (no value), jumper:SJ
- added SV1: (no value), con-harting-ml:ML6
- added SV2: (no value), con-lstb:MA04-1
- PAD1, PAD2, PAD3, PAD4, PAD5, PAD6: device wirepad:SMD2 -> wirepad:1,6/0,9
Connections:
- removed net SPI_CLK: PAD3.P
- removed net SPI_CS: PAD5.P
- removed net SPI_MISO: PAD1.P
- removed net SPI_MOSI: PAD4.P
- new net 1A: M12.P, M1A.P
- new net 1B: M11.P, M1B.P
- new net 2A: M13.P, M2A.P
- new net 2B: M14.P, M2B.P
- new net FON: 3.P, CLK.P
- new net GPIO1: IC1.(PCINT9/XTAL2)PB1, L_GPIO1.P
- new net INT: 9.P, IC1.(PCINT5/OC1B/MISO/DO/ADC5)PA5, INT.P, SV1.1
- new net M_DIR: IC1.(PCINT1/AIN0/ADC1)PA1, M8.P
- new net M_EN: IC1.(PCINT8/XTAL1/CLKI)PB0, M1.P
- new net M_MS1: M2.P, SJ1.2
- new net M_MS2: M3.P, SJ2.2
- new net M_MS3: M4.P, SJ3.2
- new net M_RESET: IC1.(PCINT7/ICP/OC0B/ADC7)PA7, M5.P
- new net M_SLEEP: IC1.(PCINT3/T0/ADC3)PA3, M6.P
- new net M_STEP: IC1.(PCINT2/AIN1/ADC2)PA2, M7.P
- new net N$9: IC1.(PCINT0/AREF/ADC0)PA0, R1.2, R2.2
- new net RESET: 5.P, IC1.(PCINT11/RESET/DW)PB3, RESET.P, SV1.5
- new net SCL: 7.P, IC1.(PCINT4/T1/SCL/USCK/ADC4)PA4, L_SCL.P, MISO41.P, SCL.P, SV1.3, SV2.2
- new net SDA: 1.P, IC1.(PCINT6/OC1A/SDA/MOSI/ADC6)PA6, L_SDA.P, MISO21.P, SDA.P, SV1.4, SV2.1
- new net U5: 4.P, C2.+, M16.P, R2.1, U5.P
- new net UCH: 6.P, UCH.P
- new net XSHUT: IC1.(PCINT10/INT0/OC0A/CKOUT)PB2, L_XSHUT.P
- net GND: now also 10.P, 8.P, C1.2, C2.-, GND.P, IC1.GND, L_GND.P, M15.P, M9.P, MISO1.P, MISO10.P, MISO11.P, MISO12.P, MISO13.P, MISO14.P, MISO15.P, MISO16.P, MISO17.P, MISO18.P, MISO19.P, MISO20.P, MISO43.P, MISO5.P, MISO6.P, MISO7.P, MISO8.P, MISO9.P, R1.1, SV1.6, SV2.4; no longer PAD6.P
- net U3.3: now also 2.P, C1.1, IC1.VCC, L_VCC.P, M10.P, MISO22.P, MISO23.P, MISO24.P, MISO25.P, MISO26.P, MISO27.P, MISO28.P, MISO29.P, MISO30.P, MISO31.P, MISO32.P, MISO33.P, MISO34.P, MISO35.P, MISO36.P, MISO37.P, MISO4.P, SJ1.1, SJ2.1, SJ3.1, SV1.2, SV2.3, U33.P; no longer PAD2.P
Other:
- moved on the sheet: PAD1, PAD2, PAD3, PAD4, PAD5, PAD6
