File: hw/zumo_uni_spi_01.brd (EAGLE design)
At the start: 100 x 80 mm, 6 parts

Commit message: added
Parts:
- added CLK, CS, GND, MISO, MISO1, MISO10, MISO11, MISO12, MISO13, MISO14, MISO15, MISO16, MISO17, MISO18, MISO19, MISO2, MISO20, MISO21, MISO22, MISO23, MISO24, MISO25, MISO26, MISO27, MISO28, MISO29, MISO3, MISO30, MISO31, MISO32, MISO33, MISO34, MISO35, MISO36, MISO37, MISO38, MISO4, MISO5, MISO6, MISO7, MISO8, MISO9, MOSI, PAD10, PAD11, PAD12, PAD13, PAD14, PAD15, PAD16, PAD17, PAD18, PAD19, PAD20, PAD21, PAD22, PAD23, PAD24, PAD25, PAD26, PAD27, PAD28, PAD29, PAD30, PAD31, PAD32, PAD33, PAD34, PAD35, PAD36, PAD37, PAD38, PAD39, PAD40, PAD41, PAD42, PAD43, PAD44, PAD45, PAD46, PAD47, PAD48, PAD49, PAD50, PAD51, PAD52, PAD53, PAD54, PAD55, PAD56, PAD57, PAD58, PAD59, PAD60, PAD61, PAD62, PAD63, PAD64, PAD65, PAD66, PAD67, PAD68, PAD69, PAD7, PAD70, PAD71, PAD72, PAD73, PAD74, PAD75, PAD76, PAD77, PAD78, PAD79, PAD8, PAD80, PAD81, PAD9, U33: (no value), wirepad:1,6/0,9
- moved PAD5 61.7 mm to (7.62, 1.27), flipped to the bottom
- moved PAD4 60.7 mm to (10.2, 1.27)
- moved PAD3 57.7 mm to (10.2, 1.27), flipped to the bottom
- moved PAD2 56.8 mm to (12.7, 1.27)
- moved PAD1 53.9 mm to (12.7, 1.27), flipped to the bottom
- moved PAD6 48.3 mm to (7.62, 1.27)
Connections:
- net GND: now also GND.1, MISO10.1, MISO11.1, MISO12.1, MISO13.1, MISO14.1, MISO15.1, MISO16.1, MISO17.1, MISO18.1, MISO19.1, MISO20.1, MISO5.1, MISO6.1, MISO7.1, MISO8.1, MISO9.1
- net SPI_CLK: now also CLK.1, MISO3.1
- net SPI_CS: now also CS.1, MISO1.1
- net SPI_MISO: now also MISO.1, MISO21.1
- net SPI_MOSI: now also MISO2.1, MOSI.1
- net U3.3: now also MISO22.1, MISO23.1, MISO24.1, MISO25.1, MISO26.1, MISO27.1, MISO28.1, MISO29.1, MISO30.1, MISO31.1, MISO32.1, MISO33.1, MISO34.1, MISO35.1, MISO36.1, MISO37.1, MISO38.1, MISO4.1, U33.1
Routing:
- net U3.3: track 0.00 -> 51.9 mm
- net GND: track 0.00 -> 51.3 mm
- net SPI_MOSI: track 0.00 -> 8.67 mm
- net SPI_CS: track 0.00 -> 8.67 mm
- net SPI_MISO: track 0.00 -> 7.62 mm
- net SPI_CLK: track 0.00 -> 7.62 mm
Other:
- board size 100 x 80 mm -> 19 x 48.9 mm
- board text added: "3.3V"
- board text added: "CLK"
- board text added: "CS"
- board text added: "GND"
- board text added: "MISO"
- board text added: "MOSI"
