File: hw/zumo_uni_spi_01.sch (EAGLE design)
At the start: 6 parts

Commit message: added
Parts:
- added CLK, CS, GND, MISO, MISO1, MISO10, MISO11, MISO12, MISO13, MISO14, MISO15, MISO16, MISO17, MISO18, MISO19, MISO2, MISO20, MISO21, MISO22, MISO23, MISO24, MISO25, MISO26, MISO27, MISO28, MISO29, MISO3, MISO30, MISO31, MISO32, MISO33, MISO34, MISO35, MISO36, MISO37, MISO38, MISO4, MISO5, MISO6, MISO7, MISO8, MISO9, MOSI, PAD10, PAD11, PAD12, PAD13, PAD14, PAD15, PAD16, PAD17, PAD18, PAD19, PAD20, PAD21, PAD22, PAD23, PAD24, PAD25, PAD26, PAD27, PAD28, PAD29, PAD30, PAD31, PAD32, PAD33, PAD34, PAD35, PAD36, PAD37, PAD38, PAD39, PAD40, PAD41, PAD42, PAD43, PAD44, PAD45, PAD46, PAD47, PAD48, PAD49, PAD50, PAD51, PAD52, PAD53, PAD54, PAD55, PAD56, PAD57, PAD58, PAD59, PAD60, PAD61, PAD62, PAD63, PAD64, PAD65, PAD66, PAD67, PAD68, PAD69, PAD7, PAD70, PAD71, PAD72, PAD73, PAD74, PAD75, PAD76, PAD77, PAD78, PAD79, PAD8, PAD80, PAD81, PAD9, U33: (no value), wirepad:1,6/0,9
Connections:
- net GND: now also GND.P, MISO10.P, MISO11.P, MISO12.P, MISO13.P, MISO14.P, MISO15.P, MISO16.P, MISO17.P, MISO18.P, MISO19.P, MISO20.P, MISO5.P, MISO6.P, MISO7.P, MISO8.P, MISO9.P
- net SPI_CLK: now also CLK.P, MISO3.P
- net SPI_CS: now also CS.P, MISO1.P
- net SPI_MISO: now also MISO.P, MISO21.P
- net SPI_MOSI: now also MISO2.P, MOSI.P
- net U3.3: now also MISO22.P, MISO23.P, MISO24.P, MISO25.P, MISO26.P, MISO27.P, MISO28.P, MISO29.P, MISO30.P, MISO31.P, MISO32.P, MISO33.P, MISO34.P, MISO35.P, MISO36.P, MISO37.P, MISO38.P, MISO4.P, U33.P
