File: hw/zumo_tb_02.brd (EAGLE design)
At the start: 99.1 x 91.4 mm, 170 parts, among them IC1 LT 1963 AEST-3.3 (1.5A), IC10 ESP32-WROVER, IC11 MCP1703DB, IC12 MCP1703DB, IC2 MCP1703DB, IC3 LM317MBSTT3, IC5 STM32G081RBT6, K1 68712414522, Q2 BSS138, Q3 BSS138, Q5 IRLML5203, U1 W25Q40BVSN

Commit message: some optimiziations
Parts:
- added H3, H4, H5, H6: MOUNT-HOLE2.8, holes:2,8
Routing:
- net BUS_FON: track 92.9 -> 36.0 mm, vias 6 -> 2
- net ESP_TXD: track 128.1 -> 144.1 mm, vias 13 -> 14
- net ESP_IO4: track 49.7 -> 64.5 mm
- net RPI_13: track 154.3 -> 169.0 mm
- net SDA: track 517.3 -> 506.3 mm, vias 31 -> 32
- net RPI_11: track 129.8 -> 139.3 mm
- net ADC0: track 36.2 -> 43.2 mm
- net SD_CMD: track 47.0 -> 53.2 mm
- net ESP_IO12_SCL: track 66.4 -> 71.7 mm
- net RPI_18: track 87.7 -> 92.3 mm
- net RPI_INT: track 93.3 -> 97.7 mm
- net RPI_RXD: track 129.7 -> 125.7 mm, vias 6 -> 8
- net SPI_CS: track 295.9 -> 299.8 mm
- net SD_DAT3: track 53.4 -> 49.9 mm
- net L_RST_5: track 77.8 -> 80.6 mm, vias 4 -> 5
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
Commit message: added
Parts:
- added D4: (no value), diode:MELF-MLL41
- added PAD21, PAD22, PAD23, PAD24: (no value), wirepad:1,6/0,8
- added PAD25: (no value), wirepad:1,6/0,9
- added SJ28: (no value), jumper:SJ
Connections:
- net N$1 renamed UCH4
- net N$10 renamed UCH5
- net N$11 renamed UCH3
- removed net U_CHARGE1: (+).1, +-.2, BUS_10.6, D1.A, D5.A
- removed net U_CHARGE2: D1.C, Q5.2, R2.2, R5.2, SJ11.3
- new net UCH: (+).1, D1.A
- new net UCH1: D1.C, PAD21.1, R2.2, SJ11.3, SJ28.2
- new net UCH2: D4.A, PAD22.1, Q5.2, R5.2, SJ28.1
- new net UCH6: +-.2, BUS_10.6, D5.A, PAD25.1
- net GND: now also PAD23.1, PAD24.1
- net VBAT: now also D4.C
Routing:
- net VBAT: track 159.3 -> 253.7 mm, vias 6 -> 8
- net U_CHARGE1: track 68.1 -> 0.00 mm, vias 1 -> 0
- net UCH6: track 0.00 -> 65.8 mm, vias 0 -> 3
- net UCH1: track 0.00 -> 59.9 mm, vias 0 -> 4
- net U_CHARGE2: track 58.2 -> 0.00 mm, vias 5 -> 0
- net UCH: track 0.00 -> 42.6 mm, vias 0 -> 2
- net UCH2: track 0.00 -> 31.8 mm, vias 0 -> 4
- net GND: track 830.4 -> 860.1 mm, vias 104 -> 122
- net SPI_CLK: track 294.7 -> 303.6 mm
- net LCD_SDA: track 94.2 -> 102.8 mm
- net CAM_D1: track 73.1 -> 77.6 mm
- net L_INT: track 313.0 -> 317.1 mm, vias 9 -> 11
- net CAM_U3.3: track 40.5 -> 44.5 mm
- net BUS_RESET: track 90.6 -> 94.3 mm
- net SCL2: track 230.5 -> 233.6 mm
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- added copper zone on layer 1, net UCH1
- added copper zone on layer 16, net UCH1
- added copper zone on layer 1, net UCH6
- added copper zone on layer 16, net UCH6
- removed copper zone on layer 1, net U_CHARGE1
- removed copper zone on layer 16, net U_CHARGE1
- removed copper zone on layer 1, net U_CHARGE2
- removed copper zone on layer 16, net U_CHARGE2
Other:
- board text added: "+"
- board text added: "-"
- board text added: "BNO055"
- board text added: "ESP32 WROVER"
- board text added: "ESP32CAM"
- board text added: "I2C"
- board text added: "IN+"
- board text added: "IN-"
- board text added: "OLED"
- board text added: "OPI"
- board text added: "RPI DISPLAY"
- board text added: "RPI Display"
- board text added: "SDCard"
- board text added: "SPI"
- board text added: "STM32"

Commit message: added
Parts:
- added C26, C27: 470uF/10V, rcl:SMC_D
- added SJ27: (no value), jumper:SJ_2
- moved SJ26 1.08 mm to (65.6, 37.2)
Connections:
- new net U5M: D2.C, SJ27.2, XV11.3
- net GND: now also C26.-, C27.-
- net U5: now also C26.+, C27.+, SJ27.1; no longer D2.C, XV11.3
- net VBAT: now also SJ27.3
Routing:
- net U5M: track 0.00 -> 32.6 mm, vias 0 -> 5
- net U5: track 230.9 -> 247.3 mm, vias 15 -> 17
- net U3.3: track 559.8 -> 566.0 mm
- net GND: track 860.1 -> 865.5 mm, vias 122 -> 150
- net SDA2: track 219.4 -> 222.0 mm
- net L_RST_3: track 81.6 -> 83.2 mm
- net VBAT: track 253.7 -> 255.3 mm
- net SPI_CS: track 299.6 -> 301.2 mm
- net FLASH_WP: track 88.6 -> 89.8 mm
- net ESP_BOOT: track 286.2 -> 287.4 mm
- net ESP_IO4: track 64.5 -> 65.1 mm
- net CAM_D2: track 126.7 -> 126.4 mm, vias 5 -> 7

Commit message: added
Connections:
- net ZUMO_VREG renamed VREG
Changed lines of the file:
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@@
 <?xml version="1.0" encoding="utf-8"?>
 <!DOCTYPE eagle SYSTEM "eagle.dtd">
-<eagle version="9.5.2">
+<eagle version="9.6.2">
 <drawing>
 <settings>
@@
 <wire x1="43.7617625" y1="87.1728" x2="42.1484875" y2="87.1728" width="0.381" layer="1"/>
 </signal>
-<signal name="ZUMO_VREG">
+<signal name="VREG">
 <contactref element="SJ8" pad="1"/>
 <contactref element="SV2" pad="10"/>
