File: hw/zumo_tb_02.sch (EAGLE design)
At the start: 170 parts, among them IC1 LT 1963 AEST-3.3 (1.5A), IC10 ESP32-WROVER, IC11 MCP1703DB, IC12 MCP1703DB, IC2 MCP1703DB, IC3 LM317MBSTT3, IC5 STM32G081RBT6, K1 68712414522, Q2 BSS138, Q3 BSS138, Q5 IRLML5203, U1 W25Q40BVSN

Commit message: some optimiziations
Parts:
- added H3, H4, H5, H6: MOUNT-HOLE2.8, holes:MOUNT-HOLE2.8
Changed lines of the file:
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@@
 <part name="PAD20" library="wirepad" library_urn="urn:adsk.eagle:library:412" deviceset="1,6/0,9" device="" package3d_urn="urn:adsk.eagle:package:30840/1"/>
 <part name="Q5" library="transistor-power" library_urn="urn:adsk.eagle:library:400" deviceset="IRLML5203" device="" package3d_urn="urn:adsk.eagle:package:29512/2"/>
+<part name="H3" library="holes" library_urn="urn:adsk.eagle:library:237" deviceset="MOUNT-HOLE" device="2.8" package3d_urn="urn:adsk.eagle:package:14271/1"/>
+<part name="H4" library="holes" library_urn="urn:adsk.eagle:library:237" deviceset="MOUNT-HOLE" device="2.8" package3d_urn="urn:adsk.eagle:package:14271/1"/>
+<part name="H5" library="holes" library_urn="urn:adsk.eagle:library:237" deviceset="MOUNT-HOLE" device="2.8" package3d_urn="urn:adsk.eagle:package:14271/1"/>
+<part name="H6" library="holes" library_urn="urn:adsk.eagle:library:237" deviceset="MOUNT-HOLE" device="2.8" package3d_urn="urn:adsk.eagle:package:14271/1"/>
 </parts>
 <sheets>
@@
 <attribute name="NAME" x="27.94" y="30.48" size="1.778" layer="95" rot="R90"/>
 <attribute name="VALUE" x="30.48" y="30.48" size="1.778" layer="96" rot="R90"/>
+</instance>
+<instance part="H3" gate="G$1" x="96.52" y="144.78" smashed="yes">
+<attribute name="NAME" x="98.552" y="145.3642" size="1.778" layer="95"/>
+<attribute name="VALUE" x="98.552" y="142.3162" size="1.778" layer="96"/>
+</instance>
+<instance part="H4" gate="G$1" x="96.52" y="137.16" smashed="yes">
+<attribute name="NAME" x="98.552" y="137.7442" size="1.778" layer="95"/>
+<attribute name="VALUE" x="98.552" y="134.6962" size="1.778" layer="96"/>
+</instance>
+<instance part="H5" gate="G$1" x="96.52" y="152.4" smashed="yes">
+<attribute name="NAME" x="98.552" y="152.9842" size="1.778" layer="95"/>
+<attribute name="VALUE" x="98.552" y="149.9362" size="1.778" layer="96"/>
+</instance>
+<instance part="H6" gate="G$1" x="96.52" y="129.54" smashed="yes">
+<attribute name="NAME" x="98.552" y="130.1242" size="1.778" layer="95"/>
+<attribute name="VALUE" x="98.552" y="127.0762" size="1.778" layer="96"/>
 </instance>
 </instances>
@@
 <pinref part="Q5" gate="G$1" pin="D"/>
 <junction x="35.56" y="25.4"/>
-<pinref part="Q5" gate="G$1" pin="D"/>
 </segment>
 </net>
@@
 <pinref part="GND41" gate="1" pin="GND"/>
 <pinref part="PAD17" gate="1" pin="P"/>
-<pinref part="PAD17" gate="1" pin="P"/>
 <wire x1="104.14" y1="248.92" x2="111.76" y2="248.92" width="0.1524" layer="91"/>

Commit message: added
Parts:
- added D4: (no value), diode:DIODE-MELF-MLL41
- added PAD21, PAD22, PAD23, PAD24: (no value), wirepad:1,6/0,8
- added PAD25: (no value), wirepad:1,6/0,9
- added SJ28: (no value), jumper:SJ
Connections:
- net N$1 renamed UCH4
- net N$10 renamed UCH5
- net N$11 renamed UCH3
- removed net U_CHARGE1: (+).P, +-.2, BUS_10.6, D1.A, D5.A
- removed net U_CHARGE2: D1.C, Q5.S, R2.2, R5.2, SJ11.3
- new net UCH: (+).P, D1.A
- new net UCH1: D1.C, PAD21.P, R2.2, SJ11.3, SJ28.2
- new net UCH2: D4.A, PAD22.P, Q5.S, R5.2, SJ28.1
- new net UCH6: +-.2, BUS_10.6, D5.A, PAD25.P
- net GND: now also PAD23.P, PAD24.P
- net VBAT: now also D4.C
Other:
- moved on the sheet: C6, D3, IC3, Q5, R12, R13, R5, R8, T1

Commit message: added
Parts:
- added C26, C27: 470uF/10V, rcl:CPOL-EUSMCD
- added SJ27: (no value), jumper:SJ2W
Connections:
- new net U5M: D2.C, SJ27.2, XV11-3.S
- net GND: now also C26.-, C27.-
- net U5: now also C26.+, C27.+, SJ27.1; no longer D2.C, XV11-3.S
- net VBAT: now also SJ27.3
Other:
- moved on the sheet: D2, LED1A, LED1B, LED2, R11, R16, R23, T2, XV11-1, XV11-2, XV11-3, XV11-4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

Commit message: added
Connections:
- net ZUMO_VREG renamed VREG
Changed lines of the file:
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@@
 <?xml version="1.0" encoding="utf-8"?>
 <!DOCTYPE eagle SYSTEM "eagle.dtd">
-<eagle version="9.5.2">
+<eagle version="9.6.2">
 <drawing>
 <settings>
@@
 </segment>
 </net>
-<net name="ZUMO_VREG" class="0">
+<net name="VREG" class="0">
 <segment>
 <pinref part="SJ8" gate="1" pin="1"/>
