Commit message: -

File: ros2_ws/src/ros2zumo_pkg/urdf/roszumo.urdf (robot description, URDF)
Before this commit: robot zumoros, 2 links, 1 joints
Links:
- added link base_footprint, mass 0.0001; visual box size=0.001 0.001 0.001
Joints:
- added joint base_footprint_joint: type fixed, parent base_footprint, child base_link, origin xyz=0 0 0.04 rpy=0 0 0
